File: V0.1/DeHisser4IEM/DeHisser4IEM.kicad_pcb (KiCad board)
At the start: 2 copper layers, 12.7 x 34.3 mm, 6 parts

Commit message: Update readme.md
Parts:
- REF** (x2): value 33k -> 33
- REF**: value 3,3 -> 3.3
Changed lines of the file:
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@@
         (effects (font (size 1 1) (thickness 0.15)))
     )
-    (fp_text value "33k" (at 0 1.65 90) (layer "F.Fab")
+    (fp_text value "33" (at 0 1.65 90) (layer "F.Fab")
         (effects (font (size 1 1) (thickness 0.15)))
     )
@@
         (effects (font (size 1 1) (thickness 0.15)))
     )
-    (fp_text value "33k" (at 0 1.65 90) (layer "F.Fab")
+    (fp_text value "33" (at 0 1.65 90) (layer "F.Fab")
         (effects (font (size 1 1) (thickness 0.15)))
     )
@@
         (effects (font (size 1 1) (thickness 0.15)))
     )
-    (fp_text value "3,3" (at 0 1.65 90) (layer "F.Fab")
+    (fp_text value "3.3" (at 0 1.65 90) (layer "F.Fab")
         (effects (font (size 1 1) (thickness 0.15)))
     )
